File: yubikey/yubikey.kicad_pcb (KiCad board)
At the start: 4 copper layers, 18.5 x 45 mm, 26 parts, among them J1 USB_C_Receptacle_USB2.0_16P, SW1 BOOTSEC, SW2 RESET, U1 ATECC608A-SSHDA, U2 RP2040, U3 W25Q128JVS, Y1 12MHz

Commit message: added some more pictures to the pcb
Parts:
- added G*** (x5): LOGO, yubico:yubico, F.Cu at (124.5, 124.0)
