File: yubikey/yubikey.kicad_sch (KiCad schematic)
At the start: 26 parts, among them J1 USB_C_Receptacle_USB2.0_16P, SW1 BOOTSEC, SW2 RESET, U1 ATECC608A-SSHDA, U2 RP2040, U3 W25Q128JVS, Y1 12MHz

Commit message: quick few updates
Connections:
- net GPI02 is gone; now on net GPIO2: SW1.2
Other:
- moved on the sheet: R6
Changed lines of the file:
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@@
 	(wire
 		(pts
-			(xy 148.59 52.07) (xy 148.59 55.88)
+			(xy 148.59 52.07) (xy 148.59 53.34)
 		)
 		(stroke
@@
 	(wire
 		(pts
+			(xy 148.59 60.96) (xy 148.59 63.5)
+		)
+		(stroke
+			(width 0)
+			(type default)
+		)
+	)
+	(wire
+		(pts
 			(xy 171.45 34.29) (xy 180.34 34.29)
 		)
@@
 		)
 	)
-	(label "GPI02"
+	(label "GPIO2"
 		(at 269.24 71.12 180)
 		(effects
@@
 	(symbol
 		(lib_id "Device:R_US")
-		(at 148.59 59.69 0)
+		(at 148.59 57.15 0)
 		(unit 1)
 		(exclude_from_sim no)
@@
 		(fields_autoplaced yes)
 		(property "Reference" "R6"
-			(at 151.13 58.4199 0)
+			(at 151.13 55.8799 0)
 			(effects
 				(font
@@
 		)
 		(property "Value" "10k"
-			(at 151.13 60.9599 0)
+			(at 151.13 58.4199 0)
 			(effects
 				(font
@@
 		)
 		(property "Footprint" "Inductor_SMD:L_0402_1005Metric"
-			(at 149.606 59.944 90)
+			(at 149.606 57.404 90)
 			(effects
 				(font
@@
 		)
 		(property "Datasheet" "~"
-			(at 148.59 59.69 0)
+			(at 148.59 57.15 0)
 			(effects
 				(font
@@
 		)
 		(property "Description" "Resistor, US symbol"
-			(at 148.59 59.69 0)
+			(at 148.59 57.15 0)
 			(effects
 				(font
